File: mixer_board_smd_full.brd (EAGLE design)
At the start: 100 x 100 mm, 71 parts, among them J1 DCJ0202, K1 G5V1, K2 G5V1, K3 G5V1, K4 TQ2-5V, P1 10k, P2 10k, P3 10k, U1 PIC16F18426

Commit message: before auto router
Routing:
- net N$29: track 24.5 -> 34.2 mm
Changed lines of the file:
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@@
 <autorouter>
 <pass name="Default">
-<param name="RoutingGrid" value="0.125mm"/>
+<param name="RoutingGrid" value="4.92125984mil"/>
 <param name="AutoGrid" value="1"/>
 <param name="Efforts" value="2"/>
 <param name="TopRouterVariant" value="1"/>
 <param name="tpViaShape" value="round"/>
-<param name="PrefDir.1" value="\"/>
+<param name="PrefDir.1" value="a"/>
 <param name="PrefDir.2" value="0"/>
 <param name="PrefDir.3" value="0"/>
@@
 <contactref element="U$16" pad="1'"/>
 <contactref element="SUMMER" pad="7"/>
-<wire x1="83.61" y1="26.035" x2="80.165" y2="26.035" width="0.3048" layer="1"/>
+<wire x1="83.61" y1="26.035" x2="81.3384" y2="26.035" width="0.3048" layer="1"/>
+<wire x1="81.28" y1="26.035" x2="80.165" y2="26.035" width="0.3048" layer="1"/>
 <wire x1="80.165" y1="26.035" x2="79.53" y2="25.4" width="0.3048" layer="1"/>
 <wire x1="79.2" y1="19.05" x2="79.53" y2="19.38" width="0.3048" layer="1"/>
 <wire x1="79.53" y1="19.38" x2="79.53" y2="25.4" width="0.3048" layer="1"/>
-<wire x1="90.96" y1="17.14" x2="90.32" y2="17.78" width="0.3048" layer="1"/>
-<wire x1="90.32" y1="17.78" x2="90.17" y2="17.78" width="0.3048" layer="1"/>
-<via x="90.17" y="17.78" extent="1-16" drill="0.35"/>
-<wire x1="90.17" y1="17.78" x2="87.63" y2="20.32" width="0.3048" layer="16"/>
+<wire x1="92.71" y1="17.78" x2="91.6" y2="17.78" width="0.3048" layer="1"/>
+<wire x1="90.96" y1="17.14" x2="91.6" y2="17.78" width="0.3048" layer="1"/>
+<via x="92.71" y="17.78" extent="1-16" drill="0.35"/>
+<wire x1="92.71" y1="17.78" x2="92.71" y2="19.05" width="0.3048" layer="16"/>
+<wire x1="92.71" y1="19.05" x2="91.44" y2="20.32" width="0.3048" layer="16"/>
+<wire x1="91.44" y1="20.32" x2="87.63" y2="20.32" width="0.3048" layer="16"/>
 <via x="87.63" y="20.32" extent="1-16" drill="0.35"/>
 <wire x1="87.63" y1="20.32" x2="87.63" y2="22.86" width="0.3048" layer="1"/>
 <via x="87.63" y="22.86" extent="1-16" drill="0.35"/>
-<via x="83.82" y="25.5956" extent="1-16" drill="0.35"/>
-<wire x1="87.726" y1="23.8470875" x2="87.726" y2="24.4129125" width="0.3048" layer="16"/>
+<via x="81.915" y="26.6116" extent="1-16" drill="0.35"/>
+<wire x1="87.726" y1="23.8470875" x2="87.726" y2="26.8656" width="0.3048" layer="16"/>
 <wire x1="87.63" y1="22.86" x2="87.63" y2="23.7510875" width="0.3048" layer="16"/>
 <wire x1="87.63" y1="23.7510875" x2="87.726" y2="23.8470875" width="0.3048" layer="16"/>
-<wire x1="87.726" y1="24.4129125" x2="86.5433125" y2="25.5956" width="0.3048" layer="16"/>
-<wire x1="86.5433125" y1="25.5956" x2="83.82" y2="25.5956" width="0.3048" layer="16"/>
-<wire x1="83.82" y1="25.5956" x2="83.61" y2="25.8056" width="0.3048" layer="1"/>
-<wire x1="83.61" y1="25.8056" x2="83.61" y2="26.035" width="0.3048" layer="1"/>
+<wire x1="87.726" y1="26.8656" x2="82.169" y2="26.8656" width="0.3048" layer="16"/>
+<wire x1="82.169" y1="26.8656" x2="81.915" y2="26.6116" width="0.3048" layer="16"/>
+<wire x1="83.61" y1="26.035" x2="82.4916" y2="26.035" width="0.3048" layer="1"/>
+<wire x1="81.915" y1="26.6116" x2="81.3384" y2="26.035" width="0.3048" layer="1"/>
+<wire x1="81.3384" y1="26.035" x2="81.28" y2="26.035" width="0.3048" layer="1"/>
 </signal>
 <signal name="N$7">
@@
 <contactref element="K3" pad="2"/>
 <contactref element="R28" pad="2"/>
+<wire x1="35.88" y1="85.09" x2="63.5" y2="95.25" width="0" layer="19" extent="1-1"/>
 <wire x1="81.34" y1="69.85" x2="63.5" y2="95.25" width="0" layer="19" extent="1-1"/>
-<wire x1="35.88" y1="85.09" x2="63.5" y2="95.25" width="0" layer="19" extent="1-1"/>
 </signal>
 <signal name="SW2">
@@
 <contactref element="U1" pad="12"/>
 <contactref element="SV1" pad="5"/>
-<wire x1="81.34" y1="73.66" x2="73.66" y2="81.28" width="0" layer="19" extent="1-1"/>
+<wire x1="73.66" y1="81.28" x2="81.34" y2="73.66" width="0" layer="19" extent="1-1"/>
 </signal>
 <signal name="N$43">

Commit message: after auto router
Routing:
- net V-: track 35.8 -> 333.3 mm, vias 0 -> 1
- net SW1: track 0.00 -> 111.9 mm
- net N$18: track 7.45 -> 116.6 mm, vias 0 -> 7
- net SW2: track 0.00 -> 96.3 mm, vias 0 -> 1
- net SW3: track 0.00 -> 86.8 mm, vias 0 -> 1
- net N$4: track 0.00 -> 79.4 mm, vias 0 -> 2
- net N$3: track 0.00 -> 75.8 mm
- net N$42: track 0.00 -> 74.1 mm, vias 0 -> 2
- net N$30: track 7.89 -> 76.8 mm
- net N$14: track 0.00 -> 66.0 mm, vias 0 -> 2
- net N$39: track 0.00 -> 64.6 mm, vias 0 -> 1
- net N$49: track 0.00 -> 57.6 mm
- net V+: track 43.3 -> 98.9 mm, vias 0 -> 3
- net SW4: track 0.00 -> 47.1 mm, vias 0 -> 1
- net N$12: track 0.00 -> 47.0 mm
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