File: mixer_board_smd_full.brd (EAGLE design)
At the start: 100 x 100 mm, 71 parts, among them J1 DCJ0202, K1 G5V1, K2 G5V1, K3 G5V1, K4 TQ2-5V, P1 10k, P2 10k, P3 10k, U1 PIC16F18426

Commit message: I think it's done
and ready to be shipped.
Parts:
- renumbered J1 to PWR, SV1 to ICSP, U$16 to GAIN, U1 to PIC16
Other:
- board text added: "PWR"

Commit message: all of the changes
Routing:
- net GND: track 753.8 -> 807.6 mm, vias 5 -> 7
Changed lines of the file:
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@@
 <?xml version="1.0" encoding="utf-8"?>
 <!DOCTYPE eagle SYSTEM "eagle.dtd">
-<eagle version="9.4.0">
+<eagle version="9.4.2">
 <drawing>
 <settings>
@@
 <layers>
 <layer number="1" name="Top" color="4" fill="1" visible="yes" active="yes"/>
+<layer number="2" name="Route2" color="1" fill="3" visible="no" active="no"/>
+<layer number="15" name="Route15" color="4" fill="6" visible="no" active="no"/>
 <layer number="16" name="Bottom" color="1" fill="1" visible="yes" active="yes"/>
 <layer number="17" name="Pads" color="2" fill="1" visible="yes" active="yes"/>
@@
 <wire x1="94.6784" y1="13.19555" x2="93.4052" y2="14.46875" width="0.3048" layer="1"/>
 <wire x1="92.71" y1="3.81" x2="94.6784" y2="5.7784" width="0.3048" layer="1"/>
+<via x="48.26" y="10.16" extent="1-16" drill="0.35"/>
+<wire x1="92.71" y1="3.81" x2="90.49374375" y2="3.81" width="0.3048" layer="1"/>
+<wire x1="54.67" y1="3.72394375" x2="54.67" y2="3.75" width="0.3048" layer="1"/>
+<wire x1="90.49374375" y1="3.81" x2="88.52534375" y2="1.8416" width="0.3048" layer="1"/>
+<wire x1="88.52534375" y1="1.8416" x2="56.55234375" y2="1.8416" width="0.3048" layer="1"/>
+<wire x1="56.55234375" y1="1.8416" x2="54.67" y2="3.72394375" width="0.3048" layer="1"/>
+<wire x1="54.67" y1="3.75" x2="48.26" y2="10.16" width="0.3048" layer="1"/>
+<wire x1="48.26" y1="10.16" x2="43.18" y2="10.16" width="0.3048" layer="16"/>
+<via x="43.18" y="10.16" extent="1-16" drill="0.35"/>
 </signal>
 <signal name="V-">

Commit message: changed a few values
Parts:
- C1, C2: value (none) -> 220uF
- C4: value 10pF -> 22pF
- F2: value PTA4553 -> 10K
- R1, R2: value (none) -> 4.7k
- R13: value 390k -> 51K
- R3: value (none) -> 330R
- R4, R5: value 51k -> 22k
Changed lines of the file:
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@@
 <?xml version="1.0" encoding="utf-8"?>
 <!DOCTYPE eagle SYSTEM "eagle.dtd">
-<eagle version="9.4.2">
+<eagle version="9.4.0">
 <drawing>
 <settings>
@@
 </autorouter>
 <elements>
-<element name="C1" library="resistor" library_urn="urn:adsk.eagle:library:348" package="E1,8-4" package3d_urn="urn:adsk.eagle:package:25825/1" value="" x="82.169" y="50.01" smashed="yes" rot="R180">
+<element name="C1" library="resistor" library_urn="urn:adsk.eagle:library:348" package="E1,8-4" package3d_urn="urn:adsk.eagle:package:25825/1" value="220uF" x="82.169" y="50.01" smashed="yes" rot="R180">
 <attribute name="NAME" x="84.61" y="50.649" size="1.27" layer="33" rot="R270"/>
 <attribute name="VALUE" x="87.479" y="53.82" size="1.27" layer="27" rot="R180"/>
@@
 <attribute name="VALUE" x="73.18" y="39.05" size="1.27" layer="27" rot="R270"/>
 </element>
-<element name="C2" library="resistor" library_urn="urn:adsk.eagle:library:348" package="E1,8-4" package3d_urn="urn:adsk.eagle:package:25825/1" value="" x="89.281" y="50.32" smashed="yes">
+<element name="C2" library="resistor" library_urn="urn:adsk.eagle:library:348" package="E1,8-4" package3d_urn="urn:adsk.eagle:package:25825/1" value="220uF" x="89.281" y="50.32" smashed="yes">
 <attribute name="NAME" x="93.19" y="49.681" size="1.27" layer="33" rot="R90"/>
 <attribute name="VALUE" x="83.971" y="46.51" size="1.27" layer="27"/>
@@
 <attribute name="VALUE" x="76.99" y="27.62" size="1.27" layer="27" rot="R270"/>
 </element>
-<element name="C4" library="resistor" library_urn="urn:adsk.eagle:library:348" package="C0805" package3d_urn="urn:adsk.eagle:package:26137/1" value="10pF" x="93.19" y="26.35" smashed="yes" rot="R270">
+<element name="C4" library="resistor" library_urn="urn:adsk.eagle:library:348" package="C0805" package3d_urn="urn:adsk.eagle:package:26137/1" value="22pF" x="93.19" y="26.35" smashed="yes" rot="R270">
 <attribute name="NAME" x="94.46" y="27.62" size="1.27" layer="33" rot="R270"/>
 <attribute name="VALUE" x="90.65" y="27.62" size="1.27" layer="27" rot="R270"/>
@@
 <attribute name="VALUE" x="15.24" y="63.5" size="1.27" layer="27" rot="R180"/>
 </element>
-<element name="R1" library="resistor" library_urn="urn:adsk.eagle:library:348" package="M0805" package3d_urn="urn:adsk.eagle:package:26079/1" value="" x="82.23" y="55.09" smashed="yes" rot="R180">
+<element name="R1" library="resistor" library_urn="urn:adsk.eagle:library:348" package="M0805" package3d_urn="urn:adsk.eagle:package:26079/1" value="4.7k" x="82.23" y="55.09" smashed="yes" rot="R180">
 <attribute name="NAME" x="79.69" y="56.36" size="1.27" layer="33" rot="R180"/>
 <attribute name="VALUE" x="83.5" y="57.63" size="1.27" layer="27" rot="R180"/>
@@
 <attribute name="VALUE" x="76.99" y="32.7" size="1.27" layer="27" rot="R270"/>
 </element>
-<element name="R13" library="resistor" library_urn="urn:adsk.eagle:library:348" package="M0805" package3d_urn="urn:adsk.eagle:package:26079/1" value="390k" x="79.53" y="37.78" smashed="yes" rot="R270">
+<element name="R13" library="resistor" library_urn="urn:adsk.eagle:library:348" package="M0805" package3d_urn="urn:adsk.eagle:package:26079/1" value="51K" x="79.53" y="37.78" smashed="yes" rot="R270">
 <attribute name="NAME" x="76.99" y="42.86" size="1.27" layer="33" rot="R270"/>
 <attribute name="VALUE" x="77.79" y="33.81" size="1.27" layer="27"/>
@@
 <attribute name="VALUE" x="51.12" y="61.75" size="1.27" layer="27"/>
 </element>
-<element name="R2" library="resistor" library_urn="urn:adsk.eagle:library:348" package="M0805" package3d_urn="urn:adsk.eagle:package:26079/1" value="" x="88.58" y="55.09" smashed="yes" rot="R180">
+<element name="R2" library="resistor" library_urn="urn:adsk.eagle:library:348" package="M0805" package3d_urn="urn:adsk.eagle:package:26079/1" value="4.7k" x="88.58" y="55.09" smashed="yes" rot="R180">
 <attribute name="NAME" x="88.58" y="57.63" size="1.27" layer="33" rot="R180"/>
 <attribute name="VALUE" x="89.85" y="57.63" size="1.27" layer="27" rot="R180"/>
@@
 <attribute name="VALUE" x="88.42" y="17.46" size="1.27" layer="27" rot="R270"/>
 </element>
-<element name="R3" library="resistor" library_urn="urn:adsk.eagle:library:348" package="R0805" package3d_urn="urn:adsk.eagle:package:26059/1" value="" x="92.39" y="65.25" smashed="yes" rot="R180">
+<element name="R3" library="resistor" library_urn="urn:adsk.eagle:library:348" package="R0805" package3d_urn="urn:adsk.eagle:package:26059/1" value="330R" x="92.39" y="65.25" smashed="yes" rot="R180">
 <attribute name="NAME" x="93.66" y="63.98" size="1.27" layer="33" rot="R180"/>
 <attribute name="VALUE" x="93.66" y="67.79" size="1.27" layer="27" rot="R180"/>
 </element>
-<element name="R4" library="resistor" library_urn="urn:adsk.eagle:library:348" package="M0805" package3d_urn="urn:adsk.eagle:package:26079/1" value="51k" x="88.58" y="33.5" smashed="yes" rot="R180">
+<element name="R4" library="resistor" library_urn="urn:adsk.eagle:library:348" package="M0805" package3d_urn="urn:adsk.eagle:package:26079/1" value="22k" x="88.58" y="33.5" smashed="yes" rot="R180">
 <attribute name="NAME" x="91.12" y="32.23" size="1.27" layer="33" rot="R180"/>
 <attribute name="VALUE" x="89.85" y="36.04" size="1.27" layer="27" rot="R180"/>
 </element>
-<element name="R5" library="resistor" library_urn="urn:adsk.eagle:library:348" package="M0805" package3d_urn="urn:adsk.eagle:package:26079/1" value="51k" x="84.14" y="33.429" smashed="yes">
+<element name="R5" library="resistor" library_urn="urn:adsk.eagle:library:348" package="M0805" package3d_urn="urn:adsk.eagle:package:26079/1" value="22k" x="84.14" y="33.429" smashed="yes">
 <attribute name="NAME" x="85.41" y="29.619" size="1.27" layer="33"/>
 <attribute name="VALUE" x="82.87" y="30.889" size="1.27" layer="27"/>
@@
 <attribute name="VALUE" x="17.78" y="2.54" size="1.27" layer="27" rot="R90"/>
 </element>
-<element name="F2" library="biblib" package="PTA4553" value="PTA4553" x="26.67" y="31.75" smashed="yes" rot="R90">
+<element name="F2" library="biblib" package="PTA4553" value="10K" x="26.67" y="31.75" smashed="yes" rot="R90">
 <attribute name="NAME" x="20.32" y="2.54" size="0.8128" layer="25" rot="R90"/>
 <attribute name="VALUE" x="34.29" y="2.54" size="1.27" layer="27" rot="R90"/>
